File: SparkFun RTK Facet - Display SD SIM.sch (EAGLE design)
At the start: 25 parts, among them J1 QWIIC_RIGHT_ANGLE, J16 microSD

Commit message: Add 22ohm to USB hub D+/D-.
Parts:
- removed J2: (no value), SparkFun-Connectors:CONN_04SMD2
- removed LOGO1: QWIIC_LOGO_CONNECTOR, SparkFun-Aesthetics:QWIIC_LOGO_CONNECTOR
- added C28: 0.1uF, SparkFun-Capacitors:0.1UF-0603-25V-(+80/-20%)
- added C8: 10uF, SparkFun-Capacitors:10UF-0603-6.3V-20%
- added D1: Green, SparkFun-LED:LED-GREEN1206-BOTTOM
- added J17: NANO_SIM, ublox:NANO_SIMWURTH
- added R5: 1k, SparkFun-Resistors:1KOHM-0603-1/10W-1%
- added U13: LIS2DH12, SparkFun-Sensors:LIS2DH12
- J1: value QWIIC_RIGHT_ANGLE -> FPC_12_0.5MM2; device SparkFun-Connectors:QWIIC_CONNECTORJS-1MM -> RTK Facet:FPC_12_0.5MM2
Connections:
- removed net SCL: J1.4, OLED1.D0/SCK
- removed net SDA: J1.3, OLED1.D1/MOSI, OLED1.D2
- new net CHARGE_LED: D1.C, J1.11
- new net ESP_21/SDA: J1.10, OLED1.D1/MOSI, OLED1.D2, U13.SDA/SDI/SDO
- new net ESP_22/SCL: J1.9, OLED1.D0/SCK, U13.SCL/SPC
- new net N$3: D1.A, R5.1
- new net VIN: J1.12, R5.2
- net 3.3V: now also C28.1, C8.1, J1.3, J1.4, U13.CS, U13.SDO/SA0, U13.VDD, U13.VDD_IO; no longer J1.2
- net GND: now also C28.2, C8.2, J1.2, U13.GND, U13.RES
- net SD_!CS!: now also J1.5; no longer J2.1
- net SD_CIPO: now also J1.8; no longer J2.4
- net SD_COPI: now also J1.6; no longer J2.2
- net SD_SCK: now also J1.7; no longer J2.3
Other:
- note added: "7-Bit unshifted I2C address: 0x19"
- note added: "Interface Selection"
- note added: "LIS2DH12 / Accelerometer"
- note added: "Placeholder. Do not populate"
- note added: "SIM"
- note removed: "1.65 <= VDD <= 3.3"
- note removed: "3.3 <= VBAT <= 4.2"
- note removed: "Interface selection"
- note removed: "Power Supply"
- note removed: "The OLED requires a 1.65-3.3V supply for its logic circuits (VDD) and a 7-7.5V supply for it's display circuitry (VCC). Fortunately, it features a charge-pump boost converter to generate a 7V supply (VCC) from 3.3-4.2V. The charge-pump input voltage is taken from the VBAT line. SJ3, closed by default, shorts the VDD and VBAT lines. This way the same supply you're using to power the logic can be b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"
- note removed: "VCC (7.0-7.5V) will be generated by on-board DC-DC converter, as long as C3 and C2 are present. It's boosted up from VBAT."
- note removed: "VCC current (Externally supplied) = 1.7-6.9mA"
- note removed: "VCC current (Internally generated) = 5.8-20.9mA"
- note removed: "VDD current < 300 uA"
- moved on the sheet: C16, C4, C6, J16, R4

Commit message: Fix errors on all 3 boards after enclosure review.
* Flip connector board completely. Mirror connectors.
* Mirror connector on SD board
* Move LED above SIM socket
* Add membrane connector to SD board
* Remove switch connector from main board
* Increase width of connector board, 2mm on each side - 54mm wide
* Move LiPo Connector north as much as possible
Parts:
- added J2: FPC_12_0.5MM2, RTK Facet:FPC_12_0.5MM2
- added S1: MOMENTARY-SWITCH-SPST-SMD-5.2MM-TALL, SparkFun-Switches:MOMENTARY-SWITCH-SPST-SMD-5.2MM-TALL
- LOGO3: value OSHW-LOGOS -> OSHW-LOGOMINI; device SparkFun-Aesthetics:OSHW-LOGOS -> SparkFun-Aesthetics:OSHW-LOGOMINI
Connections:
- new net POWER_BTN: J1.2, J2.3, J2.4, S1.2
- net CHARGE_LED: now also J2.10, J2.9
- net GND: now also J2.1, J2.2, S1.1; no longer J1.2
- net VIN: now also J2.11, J2.12
Other:
- note added: "0.66" OLED"
- note added: "Charging Indicator"
- note added: "FPC To Mainboard"
- note added: "Mecahnical placeholder. Do not populate."
- note added: "To Membrane Overlay"
- note removed: "D1 (SDAin) and D2 (SDAout) are shorted for permanent I2C mode."
- note removed: "In I2C mode, D/C sets the lower bit of the 7-bit address. Short it one way or the other. D/C I2C Address =========== 0 0x3C 1 0x3D (Default)"
- note removed: "Interface BS1 BS2 =================== SPI 0 0 I2C 1 0 8-bit (6800) 0 1 8-bit (8080) 1 1"
- note removed: "Interface Selection"
- note removed: "Placeholder. Do not populate"
- note removed: "RC delay circuit for RESET line. Used to keep pinout to standard 4-pin I2C headers and JST connectors. Pulls RESET LOW momentarily at startup then pulls HIGH once capacitor is charged after 10ms"
- note removed: "The D/C jumper should be open if SPI or parallel interfaces are used. In those interfaces this pin determines whether incoming signals are data or command."
- moved on the sheet: C1, C16, C2, C28, C3, C4, C5, C6, C7, C8, D1, J1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
