File: SparkFun RTK Facet - Main.sch (EAGLE design)
At the start: 79 parts, among them J17 3-PIN SMD, J18 QWIIC_RIGHT_ANGLE, J2 U.FL, J3 Qwiic, J4 Qwiic Right Angle, Q1 600mA/40V, Q2 MBT3904DW1T1, U1 74HC4052D, U10 MCP73833, U2 3.3V, U3 U-BLOX_ZED-F9P, U4 3.3V, U5 ESP-WROOM-32NARROW, U6 CH340C, U7 MAX17048

Commit message: Add 22ohm to USB hub D+/D-.
Parts:
- removed D3: 3A/10V/280mV, SparkFun-DiscreteSemi:DIODE-SCHOTTKY-BAT60A
- removed J11, J12, J13, J8: (no value), SparkFun-Connectors:CONN_041X04_NO_SILK_NO_POP
- removed J16, J19, J9: (no value), SparkFun-Connectors:CONN_04SMD2
- removed J17: 3-PIN SMD, SparkFun-Connectors:CONN_03JST-SMD
- removed J20: (no value), SparkFun-Connectors:CONN_021X02_NO_SILK
- removed Q1: 600mA/40V, SparkFun-DiscreteSemi:TRANS_NPN-MMBT2222AL
- added C19, C9: 18pF, SparkFun-Capacitors:18PF-0603-50V-5%
- added C20: 22uF, SparkFun-Capacitors:22UF-0603-6.3V-20%
- added C21, C22, C23, C24, C26, C28, C29: 0.1uF, SparkFun-Capacitors:0.1UF-0603-25V-5%
- added C25, C27: 1.0uF, SparkFun-Capacitors:1.0UF-0603-16V-10%-X7R
- added C8: 0.1uF, SparkFun-Capacitors:0.1UF-0603-25V-(+80/-20%)
- added D4: 250mA/100V, SparkFun-DiscreteSemi:DIODE-BAS16J
- added D7: 3A/10V/280mV, SparkFun-DiscreteSemi:DIODE-SCHOTTKY-BAT60A
- added FRAME1: FRAME-LEDGER, SparkFun-Aesthetics:FRAME-LEDGER
- added J10, J15: FPC_12_0.5MM2, RTK Facet:FPC_12_0.5MM2
- added Q3: SIL2308, SparkFun-DiscreteSemi:MOSFET_COMPLIMENTARY_PAIR-SIL2308
- added R13: 1M, SparkFun-Resistors:1MOHM-0603-1/4W-5%
- added R16, R17, R19, R21, R26: 100k, SparkFun-Resistors:100KOHM-0603-1/10W-1%
- added R22, R31: 10k, SparkFun-Resistors:10KOHM-0603-1/10W-1%
- added R24: 300k, SparkFun-Resistors:300KOHM-0603-1/10W-1%
- added R25, R32: 22, SparkFun-Resistors:22OHM-0603-1/10W-1%
- added U12: AP2112K-3.3, SparkFun-IC-Power:V_REG_AP2112K-3.3V
- added U8: USB251XB, USB251xB:USB251XB
- added Y1: 24MHz, SparkFun-Clocks:CRYSTAL-24MHZ-SMD-2.0X1.6MM
- J1: value (none) -> QWIIC_RIGHT_ANGLE; device SparkFun-Connectors:CONN_041X04_NO_SILK_NO_POP -> SparkFun-Connectors:QWIIC_CONNECTORJS-1MM
- J18: value QWIIC_RIGHT_ANGLE -> FPC_12_0.5MM2; device SparkFun-Connectors:QWIIC_CONNECTORJS-1MM -> RTK Facet:FPC_12_0.5MM2
- J3: value Qwiic -> (none); device SparkFun-Connectors:I2C_STANDARDQWIIC -> SparkFun-Connectors:CONN_01PTH_NO_SILK_YES_STOP
- J4: value Qwiic Right Angle -> (none); device SparkFun-Connectors:I2C_STANDARDQWIIC -> SparkFun-Connectors:CONN_021X02_NO_SILK
- J5: device SparkFun-Connectors:CONN_04SMD2 -> SparkFun-Connectors:JST_2MM_MALE
- J6: device SparkFun-Connectors:CONN_04SMD2 -> SparkFun-Connectors:CONN_041X04_NO_SILK_NO_POP
- R1, R18: value 1k -> 100k; device SparkFun-Resistors:1KOHM-0603-1/10W-1% -> SparkFun-Resistors:100KOHM-0603-1/10W-1%
- R11: value 330 -> 1k; device SparkFun-Resistors:330OHM-0603-1/10W-1% -> SparkFun-Resistors:1KOHM-0603-1/10W-1%
- R5: value 10k -> 12k; device SparkFun-Resistors:10KOHM-0603-1/10W-1% -> SparkFun-Resistors:12KOHM-0603-1/10W-1%
- U4: value 3.3V -> ADP160; device SparkFun-IC-Power:V_REG_AP2112K-3.3V -> SparkFun-IC-Power:ADP160
Connections:
- net ESP_16/ZED-TX01 renamed ESP_16/ZED-TXO1
- removed net 5V: C6.1, D2.C, J11.4, J17.3, U2.EN, U2.IN
- removed net ESP_12: J8.3, U5.MISO_H/IO12
- removed net ESP_13: J8.2, U5.MOSI_H/IO13
- removed net ESP_15: U5.CS0_H/IO15
- removed net ESP_2/MUX_A: U1.A, U5.IO2
- removed net ESP_32/PWR_LVL_RED: U5.XTAL_P/IO32
- removed net ESP_33/PWR_LVL_GRN: U5.XTAL_N/IO33
- removed net ESP_4/MUX_B: U1.B, U5.IO4
- removed net ESP_5: J8.4, U5.CS0_V/IO5
- removed net ESP_D_N: J16.3, U6.UD-
- removed net ESP_D_P: J16.2, U6.UD+
- removed net ESP_I35/SWITCH_BASE_SELECT: Q1.C, U5.I35
- removed net UBX_D_N: J9.3, R28.1
- removed net UBX_D_P: J9.2, R27.1
- removed net VIN: C16.1, D3.C, J16.1, J17.2, J9.1, U10.VDD
- new net ESP_12/STAT_LED: R11.2, U5.MISO_H/IO12
- new net ESP_13/POWER_CTRL: D4.A, R22.1, R24.2, U5.MOSI_H/IO13
- new net ESP_15/FAST_OFF: C20.2, Q3G1.G, R24.1, U5.CS0_H/IO15
- new net ESP_2/PERIPHERAL_POWER: R1.2, U12.EN, U5.IO2
- new net ESP_32: J6.3, U5.XTAL_P/IO32
- new net ESP_33: J6.2, U5.XTAL_N/IO33
- new net ESP_3V3: C10.1, C11.1, C4.1, C5.2, R20.2, U2.OUT, U5.3V3
- new net ESP_4/MUX_A: U1.A, U5.IO4
- new net ESP_5/MUX_B: U1.B, U5.CS0_V/IO5
- new net ESP_DM: U6.UD-, U8.USBDM_DN2
- new net ESP_DP: U6.UD+, U8.USBDP_DN2
- new net ESP_I35: J6.1, U5.I35
- new net N$10: R16.2, U8.SUSP_IND
- new net N$14: R17.2, U8.HS_IND
- new net N$19: R25.2, U8.USBDM_UP
- new net N$20: R32.2, U8.USBDP_UP
- new net N$5: R2B.1, U3.EXTINT
- new net N$6: C22.1, C23.2, Q3G1.D, Q3G2.G, R26.1
- new net N$7: C9.2, R13.2, U8.XTALIN, Y1.2
- new net N$9: R5.1, U8.RBIAS
- new net POWER_BTN: C23.1, D4.C, J3.1, J5.+, R31.1
- new net USB_!RESET: C28.1, R18.1, U8.!RESET
- new net USB_DM: J18.8, R25.1
- new net USB_DP: J18.7, R32.1
- new net VBUS_DET: C29.1, R19.2, R21.1, U8.VBUS_DET
- new net VOUT: C20.1, C27.1, C6.1, Q3G2.D, R22.2, U12.IN, U2.EN, U2.IN
- new net V_RAW: C16.1, C22.2, D2.C, D7.C, Q3G2.S, R26.2, R31.2, U10.VDD
- new net V_USB: D2.A, J10.1, J15.1, J15.2, J15.3, J15.4, R21.2
- new net ZED_DM: R28.1, U8.USBDM_DN1
- new net ZED_DP: R27.1, U8.USBDP_DN1
- new net ZED_EXTINT: R2B.2, U1.Y1
- net 3.3V: now also C25.1, C26.2, C8.1, J1.2, J10.10, J10.9, J18.5, J18.6, J4.1, R18.2, U12.OUT, U8.VDD33, U8.VDDA33; no longer C10.1, C11.1, C4.1, C5.2, J1.4, J12.4, J18.2, J3.2, J4.2, R20.2, U2.OUT, U5.3V3
- net CHG_LED: now also J10.2; no longer R1.2
- net ESP_14: now also J6.4; no longer J8.1
- net ESP_18/SD_SCK: now also J10.6; no longer J19.3
- net ESP_19/SD_CIPO: now also J10.5; no longer J19.4
- net ESP_21/SDA: now also J1.3, J10.3, J18.4, U8.SDA; no longer J18.3, J3.3, J4.3
- net ESP_22/SCL: now also J1.4, J10.4, J18.3, U8.SCL; no longer J18.4, J3.4, J4.4
- net ESP_23/SD_COPI: now also J10.7; no longer J19.2
- net ESP_25/SD_!CS!: now also J10.8; no longer J19.1
- net ESP_27/ZED_!RESET!: no longer J13.3, U1.Y1
- net ESP_I34/ZED_TX_READY: no longer J13.4
- net EXTERNAL_SERIAL1_RXI: now also J18.1; no longer J12.2, J5.1
- net EXTERNAL_SERIAL1_TXO: now also J18.2; no longer J12.3, J5.2
- net GND: now also C19.1, C21.2, C24.2, C25.2, C26.1, C27.2, C28.2, C29.2, C8.2, C9.1, J10.11, J10.12, J15.10, J15.11, J15.12, J18.11, J18.12, J5.-, Q3G1.S, R1.1, R16.1, R17.1, R19.1, R5.2, U12.GND, U8.GND, U8.TEST; no longer J11.1, J12.1, J16.4, J18.1, J20.2, J3.1, J4.1, J6.1, J6.2, J9.4, Q1.E, R5.1
- net N$15: now also C21.1, U8.PLLFILT; no longer D2.A, J17.1, R18.1
- net N$17: now also C24.1, U8.CRFILT; no longer R1.1
- net N$8: now also C19.2, R13.1, U8.XTALOUT, Y1.1; no longer Q1.B, R18.2, R5.2
- net V_BATT: now also D7.A, J15.6, J15.7, J15.8, J15.9; no longer D3.A, J20.1, J6.3, J6.4
- net ZED-RXI2: now also J18.9; no longer J11.2, J5.3
- net ZED-TXO2: now also J18.10; no longer J11.3, J5.4
- net ZED_!SAFE!: no longer J13.2
- net ZED_FENCE_STAT: no longer J1.2
- net ZED_PPS_STAT: now also J4.2; no longer J13.1, R11.2
- net ZED_RTK_STAT: no longer J1.3
Other:
- note added: "600mA Max 55uA Quiescent"
- note added: "7-bit unshifted I2C address: 0x2C"
- note added: "860nA Quiescent"
- note added: "Can we indicate all on OLED: PPS RTK Stat Bluetooth Stat HPA Base Stat Batt Stat"
- note added: "ESP32 3.3V"
- note added: "GNSS data/almanac backup: 15uA"
- note added: "Peripheral 3.3V"
- note added: "Polygon Isolation: 6mil/0.1524mm"
- note added: "Power Select"
- note added: "RF Trace Width: 13mil/0.33mm"
- note added: "Soft Power Switch"
- note added: "USB Hub"
- note added: "add 0.1 to usb detect"
- note added: "add usb inline 22"
- note added: "u-blox ZED-F9P"
- note removed: "3-way Rocker"
- note removed: "5V is not guaranteed May be 3.5-5V"
- note removed: "Can we indicate all on OLED: PPS RTK Stat Bluetooth Stat HPA Base Stat Batt Stat Charging Stat"
- note removed: "External Radio RTCM In/Out"
- note removed: "External connector to display board: Charge LED"
- note removed: "I - Rover"
- note removed: "II - Base"
- note removed: "Polygon Isolation: 8mil/0.2032mm"
- note removed: "Power"
- note removed: "RF Trace Width: 13.8mil/0.35mm"
- note removed: "Serial Config NMEA Out"
- note removed: "Stat LEDs"
- note removed: "Ublox ZED-F9P"

Commit message: Fix errors on all 3 boards after enclosure review.
* Flip connector board completely. Mirror connectors.
* Mirror connector on SD board
* Move LED above SIM socket
* Add membrane connector to SD board
* Remove switch connector from main board
* Increase width of connector board, 2mm on each side - 54mm wide
* Move LiPo Connector north as much as possible
Parts:
- removed J10: FPC_12_0.5MM2, RTK Facet:FPC_12_0.5MM2
- removed J3: (no value), SparkFun-Connectors:CONN_01PTH_NO_SILK_YES_STOP
- removed J5: (no value), SparkFun-Connectors:JST_2MM_MALE
- added J8: FPC_12_0.5MM2, RTK Facet:FPC_12_0.5MM2
Connections:
- net 3.3V: now also J8.3, J8.4; no longer J10.10, J10.9
- net CHG_LED: now also J8.11; no longer J10.2
- net ESP_18/SD_SCK: now also J8.7; no longer J10.6
- net ESP_19/SD_CIPO: now also J8.8; no longer J10.5
- net ESP_21/SDA: now also J8.10; no longer J10.3
- net ESP_22/SCL: now also J8.9; no longer J10.4
- net ESP_23/SD_COPI: now also J8.6; no longer J10.7
- net ESP_25/SD_!CS!: now also J8.5; no longer J10.8
- net GND: now also J8.1; no longer J10.11, J10.12, J5.-
- net POWER_BTN: now also J8.2; no longer J3.1, J5.+
- net V_USB: now also J8.12; no longer J10.1
Other:
- note added: "Power Button on Membrane Overlay"
Changed lines of the file:
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@@
 <part name="SUPPLY30" library="SparkFun-PowerSymbols" deviceset="3.3V" device=""/>
 <part name="GND22" library="SparkFun-PowerSymbols" deviceset="GND" device=""/>
-<part name="J10" library="RTK Facet" deviceset="FPC_12_0.5MM" device="2" value="FPC_12_0.5MM2"/>
 <part name="SUPPLY7" library="SparkFun-PowerSymbols" deviceset="V_BATT" device=""/>
 <part name="GND20" library="SparkFun-PowerSymbols" deviceset="GND" device=""/>
@@
 <part name="R31" library="SparkFun-Resistors" deviceset="10KOHM" device="-0603-1/10W-1%" value="10k"/>
 <part name="SUPPLY39" library="SparkFun-PowerSymbols" deviceset="VOUT" device=""/>
-<part name="J3" library="SparkFun-Connectors" deviceset="CONN_01" device="PTH_NO_SILK_YES_STOP"/>
 <part name="FRAME1" library="SparkFun-Aesthetics" deviceset="FRAME-LEDGER" device=""/>
-<part name="J5" library="SparkFun-Connectors" deviceset="JST_2MM_MALE" device=""/>
-<part name="GND5" library="SparkFun-PowerSymbols" deviceset="GND" device=""/>
 <part name="D7" library="SparkFun-DiscreteSemi" deviceset="DIODE-SCHOTTKY" device="-BAT60A" value="3A/10V/280mV"/>
 <part name="SUPPLY37" library="SparkFun-PowerSymbols" deviceset="V_USB" device=""/>
@@
 <part name="C29" library="SparkFun-Capacitors" deviceset="0.1UF" device="-0603-25V-5%" value="0.1uF"/>
 <part name="GND9" library="SparkFun-PowerSymbols" deviceset="GND" device=""/>
+<part name="J8" library="RTK Facet" deviceset="FPC_12_0.5MM" device="2" value="FPC_12_0.5MM2"/>
 </parts>
 <sheets>
@@
 <attribute name="VALUE" x="111.76" y="116.586" size="1.778" layer="96" align="top-center"/>
 </instance>
-<instance part="J10" gate="J1" x="101.6" y="137.16" smashed="yes">
-<attribute name="NAME" x="99.06" y="152.654" size="1.778" layer="95"/>
-<attribute name="VALUE" x="89.662" y="117.094" size="1.778" layer="96"/>
-</instance>
 <instance part="SUPPLY7" gate="G$1" x="35.56" y="139.7" smashed="yes" rot="MR0">
 <attribute name="VALUE" x="35.56" y="142.494" size="1.778" layer="96" rot="MR0" align="bottom-center"/>
@@
 <attribute name="VALUE" x="109.22" y="98.806" size="1.778" layer="96" font="vector" rot="R180"/>
 <attribute name="NAME" x="109.22" y="88.392" size="1.778" layer="95" font="vector" rot="R180"/>
+</instance>
+<instance part="J8" gate="J1" x="101.6" y="134.62" smashed="yes" rot="MR180">
+<attribute name="NAME" x="99.06" y="119.126" size="1.778" layer="95" rot="MR180"/>
+<attribute name="VALUE" x="89.662" y="154.686" size="1.778" layer="96" rot="MR180"/>
 </instance>
 </instances>
@@
 <wire x1="111.76" y1="127" x2="111.76" y2="129.54" width="0.1524" layer="91"/>
 <junction x="111.76" y="129.54"/>
-<pinref part="J10" gate="J1" pin="9"/>
-<pinref part="J10" gate="J1" pin="10"/>
+<pinref part="J8" gate="J1" pin="3"/>
+<pinref part="J8" gate="J1" pin="4"/>
 </segment>
 <segment>
@@
 <wire x1="111.76" y1="121.92" x2="111.76" y2="119.38" width="0.1524" layer="91"/>
 <pinref part="GND22" gate="1" pin="GND"/>
-<wire x1="109.22" y1="124.46" x2="111.76" y2="124.46" width="0.1524" layer="91"/>
-<wire x1="111.76" y1="124.46" x2="111.76" y2="121.92" width="0.1524" layer="91"/>
-<junction x="111.76" y="121.92"/>
-<pinref part="J10" gate="J1" pin="11"/>
-<pinref part="J10" gate="J1" pin="12"/>
+<pinref part="J8" gate="J1" pin="1"/>
 </segment>
 <segment>
@@
 <wire x1="109.22" y1="142.24" x2="114.3" y2="142.24" width="0.1524" layer="91"/>
 <label x="114.3" y="142.24" size="1.27" layer="95" xref="yes"/>
-<pinref part="J10" gate="J1" pin="4"/>
+<pinref part="J8" gate="J1" pin="9"/>
 </segment>
 <segment>
@@
 <wire x1="109.22" y1="144.78" x2="114.3" y2="144.78" width="0.1524" layer="91"/>
 <label x="114.3" y="144.78" size="1.27" layer="95" xref="yes"/>
-<pinref part="J10" gate="J1" pin="3"/>
+<pinref part="J8" gate="J1" pin="10"/>
 </segment>
 <segment>
@@
 <wire x1="109.22" y1="147.32" x2="114.3" y2="147.32" width="0.1524" layer="91"/>
 <label x="114.3" y="147.32" size="1.27" layer="95" xref="yes"/>
-<pinref part="J10" gate="J1" pin="2"/>
+<pinref part="J8" gate="J1" pin="11"/>
 </segment>
 </net>
@@
 <wire x1="109.22" y1="132.08" x2="114.3" y2="132.08" width="0.1524" layer="91"/>
 <label x="114.3" y="132.08" size="1.27" layer="95" xref="yes"/>
-<pinref part="J10" gate="J1" pin="8"/>
+<pinref part="J8" gate="J1" pin="5"/>
 </segment>
 </net>
@@
 <wire x1="109.22" y1="137.16" x2="114.3" y2="137.16" width="0.1524" layer="91"/>
 <label x="114.3" y="137.16" size="1.27" layer="95" xref="yes"/>
-<pinref part="J10" gate="J1" pin="6"/>
+<pinref part="J8" gate="J1" pin="7"/>
 </segment>
 </net>
@@
 <wire x1="109.22" y1="139.7" x2="114.3" y2="139.7" width="0.1524" layer="91"/>
 <label x="114.3" y="139.7" size="1.27" layer="95" xref="yes"/>
-<pinref part="J10" gate="J1" pin="5"/>
+<pinref part="J8" gate="J1" pin="8"/>
 </segment>
 </net>
@@
 <wire x1="109.22" y1="134.62" x2="114.3" y2="134.62" width="0.1524" layer="91"/>
 <label x="114.3" y="134.62" size="1.27" layer="95" xref="yes"/>
-<pinref part="J10" gate="J1" pin="7"/>
+<pinref part="J8" gate="J1" pin="6"/>
 </segment>
 </net>
@@
 <wire x1="119.38" y1="152.4" x2="119.38" y2="149.86" width="0.1524" layer="91"/>
 <wire x1="109.22" y1="149.86" x2="119.38" y2="149.86" width="0.1524" layer="91"/>
-<pinref part="J10" gate="J1" pin="1"/>
 <pinref part="SUPPLY18" gate="G$1" pin="V_USB"/>
+<pinref part="J8" gate="J1" pin="12"/>
 </segment>
 </net>
@@
 </segment>
 </net>
+<net name="POWER_BTN" class="0">
+<segment>
+<pinref part="J8" gate="J1" pin="2"/>
+<wire x1="109.22" y1="124.46" x2="111.76" y2="124.46" width="0.1524" layer="91"/>
+<label x="111.76" y="124.46" size="1.27" layer="95" xref="yes"/>
+</segment>
+</net>
 </nets>
 </sheet>
@@
 <text x="251.46" y="187.96" size="1.778" layer="97" align="center">7-bit unshifted I2C address: 0x2C</text>
 <text x="231.14" y="271.78" size="2.54" layer="94" rot="MR180" align="center">USB Hub</text>
+<text x="30.48" y="215.9" size="1.778" layer="97" align="center">Power Button on Membrane Overlay</text>
 </plain>
 <instances>
@@
 <instance part="SUPPLY39" gate="G$1" x="86.36" y="259.08" smashed="yes">
 <attribute name="VALUE" x="86.36" y="261.874" size="1.778" layer="96" align="bottom-center"/>
-</instance>
-<instance part="J3" gate="G$1" x="12.7" y="246.38" smashed="yes">
-<attribute name="VALUE" x="10.16" y="241.554" size="1.778" layer="96" font="vector"/>
-<attribute name="NAME" x="10.16" y="249.428" size="1.778" layer="95" font="vector"/>
 </instance>
 <instance part="FRAME1" gate="G$1" x="0" y="0" smashed="yes"/>
@@
 <attribute name="REV" x="419.1" y="6.604" size="2.7432" layer="94" font="vector"/>
 </instance>
-<instance part="J5" gate="G$1" x="15.24" y="236.22" smashed="yes" rot="R90">
-<attribute name="NAME" x="9.398" y="233.68" size="1.778" layer="95" font="vector" rot="R90"/>
-</instance>
-<instance part="GND5" gate="1" x="22.86" y="231.14" smashed="yes">
-<attribute name="VALUE" x="22.86" y="230.886" size="1.778" layer="96" align="top-center"/>
-</instance>
 <instance part="R5" gate="G$1" x="185.42" y="236.22" smashed="yes" rot="R270">
 <attribute name="NAME" x="186.944" y="236.22" size="1.778" layer="95" font="vector" rot="R270" align="bottom-center"/>
@@
 <wire x1="60.96" y1="231.14" x2="60.96" y2="228.6" width="0.1524" layer="91"/>
 <pinref part="GND52" gate="1" pin="GND"/>
-</segment>
-<segment>
-<pinref part="J5" gate="G$1" pin="-"/>
-<wire x1="20.32" y1="236.22" x2="22.86" y2="236.22" width="0.1524" layer="91"/>
-<wire x1="22.86" y1="236.22" x2="22.86" y2="233.68" width="0.1524" layer="91"/>
-<pinref part="GND5" gate="1" pin="GND"/>
 </segment>
 <segment>
@@
 <wire x1="30.48" y1="231.14" x2="30.48" y2="238.76" width="0.1524" layer="91"/>
 <junction x="30.48" y="238.76"/>
-<wire x1="30.48" y1="238.76" x2="22.86" y2="238.76" width="0.1524" layer="91"/>
-<pinref part="J3" gate="G$1" pin="1"/>
-<wire x1="20.32" y1="246.38" x2="22.86" y2="246.38" width="0.1524" layer="91"/>
-<wire x1="22.86" y1="246.38" x2="22.86" y2="238.76" width="0.1524" layer="91"/>
-<pinref part="J5" gate="G$1" pin="+"/>
-<wire x1="20.32" y1="238.76" x2="22.86" y2="238.76" width="0.1524" layer="91"/>
-<junction x="22.86" y="238.76"/>
-</segment>
-</net>
+<wire x1="30.48" y1="238.76" x2="27.94" y2="238.76" width="0.1524" layer="91"/>
+<label x="27.94" y="238.76" size="1.27" layer="95" rot="R180" xref="yes"/>
+</segment>
+</net>
