File: Hardware/SparkFun RTK Facet - Cellular.brd (EAGLE design)
At the start: 60 x 30.7 mm, 69 parts, among them IC1 SN74AVC4T774PW, J18 SARA_USB, J2 NANO_SIM, J3 U.FL, J6 DIAG, Q2 310mA/60V/1.6Ω, Q3 310mA/60V/1.6Ω, Q4 310mA/60V/1.6Ω, Q5 20V/0.2A/8MHz/1.2Ω/1Vth, Q7 310mA/60V/1.6Ω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

Commit message: Net rename to indicate inputs vs outputs
Connections:
- net LTE_CTS renamed LTE_RTSO
- net LTE_RTS renamed LTE_CTSI
- net LTE_RX renamed LTE_TXO
- net LTE_TX renamed LTE_RXI
- net SARA_CTS renamed SARA_CTSO
- net SARA_RTS renamed SARA_RTSI
- net SARA_RXD renamed SARA_RXO
- net SARA_TXD renamed SARA_TXI
Changed lines of the file:
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@@
 <wire x1="-32.85" y1="28" x2="-26.92" y2="1" width="0" layer="19" extent="1-1"/>
 </signal>
-<signal name="SARA_RTS">
+<signal name="SARA_RTSI">
 <contactref element="U1" pad="10"/>
 <contactref element="TP4" pad="P$1"/>
 <contactref element="IC1" pad="6"/>
+<wire x1="29" y1="-12" x2="28.9" y2="9.05" width="0" layer="19" extent="1-1"/>
 <wire x1="-0.025" y1="-27.9" x2="29" y2="-12" width="0" layer="19" extent="1-1"/>
-<wire x1="28.9" y1="9.05" x2="-0.025" y2="-27.9" width="0" layer="19" extent="1-1"/>
 </signal>
-<signal name="SARA_CTS">
+<signal name="SARA_CTSO">
 <contactref element="U1" pad="11"/>
 <contactref element="TP3" pad="P$1"/>
 <contactref element="IC1" pad="5"/>
+<wire x1="29" y1="-15" x2="30" y2="9.05" width="0" layer="19" extent="1-1"/>
 <wire x1="-0.675" y1="-27.9" x2="29" y2="-15" width="0" layer="19" extent="1-1"/>
-<wire x1="30" y1="9.05" x2="-0.675" y2="-27.9" width="0" layer="19" extent="1-1"/>
 </signal>
-<signal name="SARA_TXD">
+<signal name="SARA_TXI">
 <contactref element="TP2" pad="P$1"/>
 <contactref element="IC1" pad="4"/>
@@
 <wire x1="-1.325" y1="-27.9" x2="29" y2="-18" width="0" layer="19" extent="1-1"/>
 </signal>
-<signal name="SARA_RXD">
+<signal name="SARA_RXO">
 <contactref element="TP1" pad="P$1"/>
 <contactref element="IC1" pad="3"/>
@@
 <wire x1="-5.58" y1="-7" x2="-5.4318" y2="-14" width="0" layer="19" extent="1-1"/>
 </signal>
-<signal name="LTE_TX">
+<signal name="LTE_RXI">
 <contactref element="TP6" pad="P$1"/>
 <contactref element="IC1" pad="13"/>
@@
 <wire x1="-1.325" y1="-22.1" x2="29" y2="-6" width="0" layer="19" extent="1-1"/>
 </signal>
-<signal name="LTE_CTS">
+<signal name="LTE_RTSO">
 <contactref element="TP7" pad="P$1"/>
 <contactref element="IC1" pad="12"/>
@@
 <wire x1="33" y1="-33" x2="-0.675" y2="-22.1" width="0" layer="19" extent="1-1"/>
 </signal>
-<signal name="LTE_RTS">
+<signal name="LTE_CTSI">
 <contactref element="TP8" pad="P$1"/>
 <contactref element="R19" pad="2"/>
@@
 <wire x1="-0.025" y1="-22.1" x2="26" y2="-19.15" width="0" layer="19" extent="1-1"/>
 </signal>
-<signal name="LTE_RX">
+<signal name="LTE_TXO">
 <contactref element="TP5" pad="P$1"/>
 <contactref element="IC1" pad="14"/>
