File: Hardware/Display/SparkFun RTK Facet - Display SD SIM.brd (EAGLE design)
At the start: 50 x 22 mm, 42 parts, among them J1 FPC_12_0.5MM_BACKFLIP, J16 microSD, J3 FPC_12_0.5MM_BACKFLIP, U13 LIS2DH12

Commit message: Increase height 2mm to 23. Move OLED connector up 1mm. Move overlay connector down.
Parts:
- U$5: device output:SIM2 -> output:RTK5#SVG0
- moved U$5 18.3 mm to (17.0, 16.0)
- moved U$7 15.8 mm to (21.0, 3.00)
- moved JP3 14.7 mm to (24.0, 3.00), turned to 0 degrees
- moved LOGO3 7.07 mm to (8.00, 3.00)
- moved C5 5.10 mm to (15.0, 5.00), turned to 270 degrees
- moved C1 4.47 mm to (12.0, 5.00), turned to 270 degrees
- moved U$3 3.10 mm to (26.3, 1.00)
- moved U$4 3.00 mm to (22.0, 1.00)
- moved OLED1 1.00 mm to (25.0, 9.70)
- moved C16 0.20 mm to (30.0, 2.80)
- moved R4 0.20 mm to (32.0, 2.80)
- moved C2 0.19 mm to (30.0, 6.00), turned to 90 degrees
- moved C6 0.19 mm to (28.0, 6.00)
- moved C7 0.19 mm to (26.0, 6.00)
- moved R2 0.19 mm to (22.0, 6.00)
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Routing:
- net 3.3V: track 0.00 -> 76.6 mm, vias 0 -> 1
- net ESP_21/SDA: track 0.00 -> 43.8 mm, vias 0 -> 4
- net POWER_BTN: track 0.00 -> 40.2 mm, vias 0 -> 2
- net CHARGE_LED: track 0.00 -> 37.1 mm, vias 0 -> 3
- net ESP_22/SCL: track 0.00 -> 35.6 mm, vias 0 -> 4
- net SD_!CS!: track 0.00 -> 34.0 mm
- net V_USB: track 0.00 -> 28.5 mm
- net SD_COPI: track 0.00 -> 16.9 mm, vias 0 -> 2
- net SD_SCK: track 0.00 -> 14.3 mm
- net SD_CIPO: track 0.00 -> 13.6 mm
- net VCC: track 0.00 -> 11.3 mm, vias 0 -> 1
- net D/C: track 0.00 -> 11.0 mm, vias 0 -> 2
- net RESET: track 0.00 -> 10.5 mm, vias 0 -> 1
- net VCOMH: track 0.00 -> 9.42 mm, vias 0 -> 1
- net N$2: track 0.00 -> 7.71 mm, vias 0 -> 1
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Other:
- board size 50 x 22 mm -> 50 x 23 mm
- board text removed: "Invert overlay connections"
- board text removed: "Move overlay connector way down"
