File: Hardware/Display/SparkFun RTK Facet - Display SD SIM.sch (EAGLE design)
At the start: 30 parts, among them J1 FPC_12_0.5MM_BACKFLIP, J16 microSD, J3 FPC_12_0.5MM_BACKFLIP, U13 LIS2DH12

Commit message: Change to push push socket on cellular board.
Parts:
- removed J16: microSD, SparkFun-Connectors:MICRO-SD-SDIOPUSH-PUSH
- added J2: MICRO-SD-PUSH-PUSH-EXT-PIN, SparkFun-Connectors:MICRO-SD-PUSH-PUSH-EXT-PIN
Connections:
- net 3.3V: now also J2.VCC; no longer J16.VCC
- net GND: now also J2.DET, J2.GND; no longer J16.GND, J16.SHIELD
- net SD_!CS!: now also J2.DAT3/!CS!; no longer J16.DAT3/!CS!
- net SD_CIPO: now also J2.DAT0/SDO; no longer J16.DAT0/SDO
- net SD_COPI: now also J2.CMD/SDI; no longer J16.CMD/SDI
- net SD_SCK: now also J2.CLK/SCK; no longer J16.CLK/SCK
Changed lines of the file:
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@@
 <layer number="56" name="wert" color="7" fill="1" visible="no" active="no"/>
 <layer number="57" name="tCAD" color="7" fill="1" visible="no" active="no"/>
+<layer number="58" name="bCAD" color="7" fill="1" visible="no" active="no"/>
 <layer number="59" name="tCarbon" color="7" fill="1" visible="no" active="no"/>
 <layer number="60" name="bCarbon" color="7" fill="1" visible="no" active="no"/>
@@
 <layer number="250" name="Descript" color="7" fill="1" visible="yes" active="yes"/>
 <layer number="251" name="SMDround" color="7" fill="1" visible="yes" active="yes"/>
+<layer number="253" name="Extra" color="7" fill="1" visible="no" active="no"/>
 <layer number="254" name="cooling" color="7" fill="1" visible="yes" active="yes"/>
 <layer number="255" name="routoute" color="7" fill="1" visible="yes" active="yes"/>
@@
 <part name="R4" library="SparkFun-Resistors" deviceset="100KOHM" device="-0603-1/10W-1%" value="100k"/>
 <part name="SUPPLY28" library="SparkFun-PowerSymbols" deviceset="3.3V" device=""/>
-<part name="J16" library="SparkFun-Connectors" deviceset="MICRO-SD-SDIO" device="PUSH-PUSH" value="microSD"/>
 <part name="SUPPLY13" library="SparkFun-PowerSymbols" deviceset="3.3V" device=""/>
 <part name="SUPPLY14" library="SparkFun-PowerSymbols" deviceset="3.3V" device=""/>
@@
 <part name="SUPPLY8" library="SparkFun-PowerSymbols" deviceset="3.3V" device=""/>
 <part name="GND5" library="SparkFun-PowerSymbols" deviceset="GND" device=""/>
-<part name="S1" library="SparkFun-Switches" deviceset="MOMENTARY-SWITCH-SPST" device="-SMD-5.2MM-TALL" value=""/>
+<part name="S1" library="SparkFun-Switches" deviceset="MOMENTARY-SWITCH-SPST" device="-SMD-5.2MM-TALL" value="MOMENTARY-SWITCH-SPST-SMD-5.2MM-TALL"/>
 <part name="GND6" library="SparkFun-PowerSymbols" deviceset="GND" device=""/>
 <part name="SUPPLY10" library="SparkFun-PowerSymbols" deviceset="V_USB" device=""/>
@@
 <part name="SUPPLY4" library="SparkFun-PowerSymbols" deviceset="V_USB" device=""/>
 <part name="J3" library="RTK Facet" deviceset="FPC_12_0.5MM" device="_BACKFLIP" value="FPC_12_0.5MM_BACKFLIP"/>
+<part name="J2" library="SparkFun-Connectors" deviceset="MICRO-SD" device="-PUSH-PUSH-EXT-PIN"/>
 </parts>
 <sheets>
@@
 <attribute name="VALUE" x="180.34" y="180.594" size="1.778" layer="96" align="bottom-center"/>
 </instance>
-<instance part="J16" gate="G$1" x="198.12" y="154.94" smashed="yes">
-<attribute name="NAME" x="193.04" y="168.148" size="1.778" layer="95"/>
-<attribute name="VALUE" x="193.04" y="139.7" size="1.778" layer="96"/>
-</instance>
 <instance part="SUPPLY13" gate="G$1" x="5.08" y="167.64" smashed="yes">
 <attribute name="VALUE" x="5.08" y="170.434" size="1.778" layer="96" align="bottom-center"/>
@@
 <attribute name="NAME" x="104.14" y="78.994" size="1.778" layer="95"/>
 <attribute name="VALUE" x="94.742" y="43.434" size="1.778" layer="96"/>
+</instance>
+<instance part="J2" gate="J1" x="198.12" y="154.94" smashed="yes">
+<attribute name="NAME" x="193.04" y="168.148" size="1.778" layer="95"/>
+<attribute name="VALUE" x="193.04" y="139.7" size="1.778" layer="96"/>
 </instance>
 </instances>
@@
 <wire x1="190.5" y1="144.78" x2="187.96" y2="144.78" width="0.1524" layer="91"/>
 <junction x="187.96" y="144.78"/>
-<pinref part="J16" gate="G$1" pin="GND"/>
-<pinref part="J16" gate="G$1" pin="SHIELD"/>
+<pinref part="J2" gate="J1" pin="GND"/>
+<pinref part="J2" gate="J1" pin="DET"/>
 </segment>
 <segment>
@@
 <wire x1="187.96" y1="165.1" x2="187.96" y2="167.64" width="0.1524" layer="91"/>
 <pinref part="SUPPLY26" gate="G$1" pin="3.3V"/>
-<pinref part="J16" gate="G$1" pin="VCC"/>
+<pinref part="J2" gate="J1" pin="VCC"/>
 </segment>
 <segment>
@@
 <wire x1="180.34" y1="165.1" x2="180.34" y2="162.56" width="0.1524" layer="91"/>
 <junction x="180.34" y="162.56"/>
-<pinref part="J16" gate="G$1" pin="DAT3/!CS!"/>
+<pinref part="J2" gate="J1" pin="DAT3/!CS!"/>
 </segment>
 <segment>
@@
 <wire x1="190.5" y1="152.4" x2="187.96" y2="152.4" width="0.1524" layer="91"/>
 <label x="187.96" y="152.4" size="1.27" layer="95" rot="R180" xref="yes"/>
-<pinref part="J16" gate="G$1" pin="CLK/SCK"/>
+<pinref part="J2" gate="J1" pin="CLK/SCK"/>
 </segment>
 <segment>
@@
 <wire x1="190.5" y1="154.94" x2="187.96" y2="154.94" width="0.1524" layer="91"/>
 <label x="187.96" y="154.94" size="1.27" layer="95" rot="R180" xref="yes"/>
-<pinref part="J16" gate="G$1" pin="DAT0/SDO"/>
+<pinref part="J2" gate="J1" pin="DAT0/SDO"/>
 </segment>
 <segment>
@@
 <wire x1="190.5" y1="149.86" x2="187.96" y2="149.86" width="0.1524" layer="91"/>
 <label x="187.96" y="149.86" size="1.27" layer="95" rot="R180" xref="yes"/>
-<pinref part="J16" gate="G$1" pin="CMD/SDI"/>
-</segment>
-<segment>
+<pinref part="J2" gate="J1" pin="CMD/SDI"/>
+</segment>
+<segment>
