File: Hardware/Connector/SparkFun RTK Facet - External Connector.sch (EAGLE design)
At the start: 22 parts, among them J1 FPC_12_0.5MM_BACKFLIP, J4 Qwiic, J5 u-blox USB, J6 FPC_12_0.5MM_BACKFLIP

Commit message: Add revisions to schematics. Add PDFs of schematics.
Other:
- note added: "N. Seidle"
- note added: "v12"
- note removed: "v10"
Changed lines of the file:
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@@
 <sheet>
 <plain>
-<text x="240.284" y="7.366" size="2.54" layer="94">v10</text>
+<text x="240.284" y="7.366" size="2.54" layer="94">v12</text>
 <text x="43.18" y="177.8" size="2.54" layer="94" rot="MR180" align="center">USB / Power</text>
 <text x="163.322" y="173.482" size="2.54" layer="94" rot="MR180" align="center">External Radio
@@
 <wire x1="195.58" y1="91.44" x2="195.58" y2="35.56" width="0.2032" layer="97" style="longdash"/>
 <wire x1="93.98" y1="91.44" x2="195.58" y2="91.44" width="0.2032" layer="97" style="longdash"/>
+<text x="171.196" y="11.176" size="2.54" layer="94">N. Seidle</text>
 </plain>
 <instances>
@@
 <attribute name="LAST_DATE_TIME" x="160.02" y="1.27" size="2.54" layer="94" font="vector"/>
 <attribute name="SHEET" x="233.68" y="1.27" size="2.54" layer="94" font="vector"/>
-<attribute name="DRAWING_NAME" x="162.814" y="17.78" size="2.7432" layer="94" font="vector"/>
+<attribute name="DRAWING_NAME" x="162.814" y="17.78" size="2.286" layer="94" font="vector"/>
 <attribute name="DESIGNER" x="170.434" y="11.176" size="2.7432" layer="94" font="vector"/>
 <attribute name="REV" x="236.22" y="6.604" size="2.7432" layer="94" font="vector"/>
@@
 <instance part="J1" gate="J1" x="111.76" y="60.96" smashed="yes" rot="MR180">
 <attribute name="NAME" x="109.22" y="45.466" size="1.778" layer="95" rot="MR180"/>
-<attribute name="VALUE" x="99.06" y="81.28" size="1.778" layer="96" rot="MR180"/>
+<attribute name="VALUE" x="106.68" y="45.72" size="1.778" layer="96" rot="MR90"/>
 </instance>
 <instance part="J6" gate="J1" x="152.4" y="60.96" smashed="yes" rot="MR180">
 <attribute name="NAME" x="149.86" y="45.466" size="1.778" layer="95" rot="MR180"/>
-<attribute name="VALUE" x="139.7" y="81.28" size="1.778" layer="96" rot="MR180"/>
+<attribute name="VALUE" x="147.574" y="45.466" size="1.778" layer="96" rot="MR90"/>
 </instance>
 </instances>
