File: Hardware/Main-LBand/SparkFun RTK Facet L-Band - Main.brd (EAGLE design)
At the start: 59.5 x 43 mm, 153 parts, among them J1 QWIIC_RIGHT_ANGLE, J2 U.FL, J9 CORTEX_JTAG_DEBUG_PTH, Q2 MBT3904DW1T1, Q3 SIL2308, U1 74HC4052D, U10 MCP73833MSOP, U12 AP2112K-3.3V, U13 POWER-DIVIDER, U2 AP2112K-3.3V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

Commit message: Update ID resistors.
Parts:
- R33: value 100k -> 1k
- R34: value 10k -> 4.7k
Changed lines of the file:
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@@
 <setting verticaltext="up"/>
 </settings>
-<grid distance="1" unitdist="mm" unit="mm" style="lines" multiple="1" display="yes" altdistance="0.1" altunitdist="mm" altunit="mm"/>
+<grid distance="0.05" unitdist="inch" unit="inch" style="lines" multiple="1" display="yes" altdistance="0.005" altunitdist="inch" altunit="inch"/>
 <layers>
 <layer number="1" name="Top/Horz" color="4" fill="1" visible="yes" active="yes"/>
-<layer number="2" name="GND/Horz" color="1" fill="3" visible="yes" active="yes"/>
-<layer number="15" name="3.3V/Vert" color="4" fill="6" visible="yes" active="yes"/>
+<layer number="2" name="GND/Horz" color="1" fill="3" visible="no" active="yes"/>
+<layer number="15" name="3.3V/Vert" color="4" fill="6" visible="no" active="yes"/>
 <layer number="16" name="Bottom/Vert" color="1" fill="1" visible="yes" active="yes"/>
 <layer number="17" name="Pads" color="2" fill="1" visible="yes" active="yes"/>
@@
 <layer number="44" name="Drills" color="7" fill="1" visible="no" active="yes"/>
 <layer number="45" name="Holes" color="7" fill="1" visible="yes" active="yes"/>
-<layer number="46" name="Milling" color="3" fill="1" visible="yes" active="yes"/>
+<layer number="46" name="Milling" color="3" fill="1" visible="no" active="yes"/>
 <layer number="47" name="Measures" color="7" fill="1" visible="no" active="yes"/>
 <layer number="48" name="Document" color="7" fill="1" visible="no" active="yes"/>
@@
 <attribute name="VALUE" x="0.0362" y="20.8288" size="0.6096" layer="27" font="vector" ratio="20" rot="R270"/>
 </element>
-<element name="R33" library="SparkFun-Resistors" package="0603" value="100k" x="3.75" y="9" smashed="yes" rot="R90">
+<element name="R33" library="SparkFun-Resistors" package="0603" value="1k" x="3.75" y="9" smashed="yes" rot="R90">
 <attribute name="NAME" x="2.988" y="9" size="0.6096" layer="25" font="vector" ratio="20" rot="R90" align="bottom-center"/>
-<attribute name="PROD_ID" value="RES-07828" x="3.75" y="9" size="1.778" layer="27" font="vector" ratio="15" rot="R90" display="off"/>
-<attribute name="VALUE" value="100k" x="4.512" y="9" size="0.6096" layer="27" font="vector" ratio="20" rot="R90" align="top-center"/>
-</element>
-<element name="R34" library="SparkFun-Resistors" package="0603" value="10k" x="3.75" y="13" smashed="yes" rot="R90">
+<attribute name="PROD_ID" value="RES-07856" x="3.75" y="9" size="1.778" layer="27" font="vector" ratio="15" rot="R90" display="off"/>
+<attribute name="VALUE" value="1k" x="4.512" y="9" size="0.6096" layer="27" font="vector" ratio="20" rot="R90" align="top-center"/>
+</element>
+<element name="R34" library="SparkFun-Resistors" package="0603" value="4.7k" x="3.75" y="13" smashed="yes" rot="R90">
 <attribute name="NAME" x="2.988" y="13" size="0.6096" layer="25" font="vector" ratio="20" rot="R90" align="bottom-center"/>
-<attribute name="PROD_ID" value="RES-00824" x="3.75" y="13" size="1.778" layer="27" font="vector" ratio="15" rot="R90" display="off"/>
-<attribute name="VALUE" x="4.512" y="13" size="0.6096" layer="27" font="vector" ratio="20" rot="R90" align="top-center"/>
+<attribute name="PROD_ID" value="RES-07857" x="3.75" y="13" size="1.778" layer="27" font="vector" ratio="15" rot="R90" display="off"/>
+<attribute name="VALUE" value="4.7k" x="4.512" y="13" size="0.6096" layer="27" font="vector" ratio="20" rot="R90" align="top-center"/>
 </element>
 <element name="U$11" library="output" package="RTK_FACET0" value="" x="44.2" y="3.175" smashed="yes"/>
