File: Hardware/Connector/KiCad/SparkFun RTK Facet - External Connector.kicad_pcb (KiCad board)
At the start: 4 copper layers, 53 x 23 mm, 38 parts, among them J1 Conn_01x12_FPC_0.5mm, J11 Conn_01x04, J12 Conn_01x04, J2 JST_Locking_4, J3 Conn_01x12_FPC_0.5mm, J4 Qwiic, J5 USB_C_Receptacle, J9 JST_Locking_4

Commit message: Add route out text
Other:
- board text added: "ROUTE OUT"
Changed lines of the file:
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@@
 				(font
 					(size 0.001 0.001)
+					(thickness 0.15)
 				)
 			)
@@
 				(font
 					(size 0.001 0.001)
+					(thickness 0.15)
 				)
 			)
@@
 				(font
 					(size 0.001 0.001)
+					(thickness 0.15)
 				)
 			)
@@
 				(font
 					(size 0.001 0.001)
+					(thickness 0.15)
 				)
 			)
@@
 		(tags "SparkFun FPC Back flip SMD")
 		(property "Reference" "J3"
-			(at 0 2.6 360)
+			(at 0 2.6 0)
 			(layer "F.Fab")
 			(effects
@@
 		)
 		(property "Value" "Conn_01x12_FPC_0.5mm"
-			(at 0 3.4 360)
+			(at 0 3.4 0)
 			(layer "F.Fab")
 			(effects
@@
 		(fp_arc
 			(start 3.62 1.55)
-			(mid 3.555421 1.692445)
+			(mid 3.555421 1.692441)
 			(end 3.409999 1.749999)
 			(stroke
@@
 		)
 		(fp_text user "Ribbon Insert"
-			(at 0 3.25 360)
+			(at 0 3.25 0)
 			(layer "F.Fab")
 			(effects
@@
 				(font
 					(size 0.001 0.001)
+					(thickness 0.15)
 				)
 			)
@@
 				(font
 					(size 0.001 0.001)
+					(thickness 0.15)
 				)
 			)
@@
 				(font
 					(size 0.001 0.001)
+					(thickness 0.15)
 				)
 			)
@@
 				(font
 					(size 0.001 0.001)
+					(thickness 0.15)
 				)
 			)
@@
 				(font
 					(size 0.001 0.001)
+					(thickness 0.15)
 				)
 			)
@@
 				(font
 					(size 0.001 0.001)
+					(thickness 0.15)
 				)
 			)
@@
 				(font
 					(size 0.001 0.001)
+					(thickness 0.15)
 				)
 			)
@@
 				(font
 					(size 0.001 0.001)
+					(thickness 0.15)
 				)
 			)
@@
 				(font
 					(size 0.001 0.001)
+					(thickness 0.15)
 				)
 			)
@@
 				(font
 					(size 0.001 0.001)
+					(thickness 0.15)
 				)
 			)
@@
 				(font
 					(size 0.001 0.001)
+					(thickness 0.15)
 				)
 			)
@@
 				(font
 					(size 0.001 0.001)
+					(thickness 0.15)
 				)
 			)
@@
 				(font
 					(size 0.001 0.001)
+					(thickness 0.15)
 				)
 			)
@@
 				(font
 					(size 0.001 0.001)
+					(thickness 0.15)
 				)
 			)
@@
 				(font
 					(size 0.001 0.001)
+					(thickness 0.15)
 				)
 			)
@@
 				(font
 					(size 0.001 0.001)
+					(thickness 0.15)
 				)
 			)
@@
 		(fp_arc
 			(start 3.62 1.55)
-			(mid 3.555421 1.692445)
+			(mid 3.555421 1.692441)
 			(end 3.409999 1.749999)
 			(stroke
@@
 				(font
 					(size 0.001 0.001)
+					(thickness 0.15)
 				)
 			)
@@
 				(font
 					(size 0.001 0.001)
+					(thickness 0.15)
 				)
 			)
@@
 		(tags "SparkFun")
 		(property "Reference" "F3"
-			(at 0 -1.397 360)
+			(at 0 -1.397 0)
 			(layer "F.Fab")
 			(effects
@@
 		)
 		(property "Value" "6V/2.0A/4.0A"
-			(at 0 1.397 360)
+			(at 0 1.397 0)
 			(layer "F.Fab")
 			(effects
@@
 				(font
 					(size 0.001 0.001)
+					(thickness 0.15)
 				)
 			)
@@
 				(font
 					(size 0.001 0.001)
+					(thickness 0.15)
 				)
 			)
@@
 				(font
 					(size 0.001 0.001)
+					(thickness 0.15)
 				)
 			)
@@
 				(font
 					(size 0.001 0.001)
+					(thickness 0.15)
 				)
 			)
@@
 				(font
 					(size 0.001 0.001)
+					(thickness 0.15)
 				)
 			)
@@
 				(font
 					(size 0.001 0.001)
+					(thickness 0.15)
 				)
 			)
@@
 				(font
 					(size 0.001 0.001)
+					(thickness 0.15)
 				)
 				(justify mirror)
@@
 				(font
 					(size 0.001 0.001)
+					(thickness 0.15)
 				)
 				(justify mirror)
@@
 				(font
 					(size 0.001 0.001)
+					(thickness 0.15)
 				)
 				(justify mirror)
@@
 				(font
 					(size 0.001 0.001)
+					(thickness 0.15)
 				)
 				(justify mirror)
@@
 				(font
 					(size 0.001 0.001)
+					(thickness 0.15)
 				)
 				(justify mirror)
@@
 				(font
 					(size 0.001 0.001)
+					(thickness 0.15)
 				)
 				(justify mirror)
@@
 			(layer "B.SilkS")
 		)
-		(group ""
-			(members "0adab0a5-48a4-499b-8b2d-36f7cf6b15ad" "4c61aae4-191b-445f-ad44-e1673ead8ec7"
-				"56663aed-dda1-412d-bb6a-b9e946c7f40d" "5d0bdac3-2d23-4a7d-8e3d-ffaee66b518f"
-				"63cfe6a6-6c19-4291-8554-338ce3b6699d" "a71a1909-78b9-425b-9d0f-e625cfee3485"
-				"af2d4dc2-88e7-48eb-9aba-13d60ff75ebd" "e3f7cf2d-54a9-4cd9-8373-3f5b4cf7dc74"
-			)
-		)
 	)
 	(gr_line
@@
 			)
 		)
+	)
+	(gr_text "ROUTE OUT"
+		(at 153.08941 94.782397 0)
+		(layer "Edge.Cuts")
+		(effects
+			(font
+				(size 1 1)
+				(thickness 0.15)
+			)
+		)
